File: easy home electronics.kicad_pcb (KiCad board)
At the start: 2 copper layers, 69.9 x 69.6 mm, 110 parts, among them J1 Screw_Terminal_01x01, J2 Screw_Terminal_01x01, J3 Screw_Terminal_01x01, J4 Conn_01x04_Pin, Q1 NPN, Q2 NPN, Q3 PMOS, Q4 NPN, Q5 BTA16-600B, Q6 NPN, SW1 SW_Push, SW2 SW_Push, SW3 SW_Push, U1 LM1117DT-3.3, U2 L78M05ABDT-TR, U3 ESP32-WROOM-32, U4 L78M05ABDT-TR, U5 PC817, U6 TLV9001IDCK, U7 ACS712xLCTR-20A, U8 HCNR200-500E

Commit message: Add files via upload
new design backup
Parts:
- removed C15: 22uf, Capacitor_SMD:C_1812_4532Metric
- removed C16: 0.1uf, Capacitor_SMD:C_1812_4532Metric
- removed C17: 1nf, Capacitor_SMD:C_1812_4532Metric
- removed D5, D6, D7: WS2812B, LED_SMD:LED_WS2812B_PLCC4_5.0x5.0mm_P3.2mm
- removed JP1, JP2: SolderJumper_2_Open, Jumper:SolderJumper-2_P1.3mm_Open_RoundedPad1.0x1.5mm
- removed Q2, Q4, Q6: NPN, Package_TO_SOT_SMD:SOT-23_Handsoldering
- removed Q3: PMOS, Package_TO_SOT_SMD:SOT-23_Handsoldering
- removed Q5: BTA16-600B, Package_TO_SOT_THT:TO-220-3_Vertical
- removed R19, R26: 22K, Resistor_SMD:R_1812_4532Metric_Pad1.30x3.40mm_HandSolder
- removed R20: 100k, Resistor_SMD:R_1812_4532Metric_Pad1.30x3.40mm_HandSolder
- removed R24, R28: 2.2K, Resistor_SMD:R_1812_4532Metric_Pad1.30x3.40mm_HandSolder
- removed R25: LDR07, OptoDevice:R_LDR_5.1x4.3mm_P3.4mm_Vertical
- removed R27, R5: 4.7k, Resistor_SMD:R_1812_4532Metric_Pad1.30x3.40mm_HandSolder
- removed R4: 10k, Resistor_SMD:R_1812_4532Metric_Pad1.30x3.40mm_HandSolder
- removed the REF** at (220.8, 44.5)
- removed the REF** at (167.0, 109.2)
- removed the REF** at (166.8, 44.5)
- removed SW1, SW2: SW_Push, Button_Switch_THT:SW_PUSH_6mm_H5mm
- removed TP14: TestPoint, TestPoint:TestPoint_Pad_D2.5mm
- removed TP17, TP18, TP19, TP20, TP21, TP22, TP23, TP24, TP25, TP26, TP27, TP28, TP29, TP30: TestPoint, TestPoint:TestPoint_Pad_D4.0mm
- removed U8: HCNR200-500E, Package_DIP:DIP-8_W7.62mm
- added H1: MountingHole_Pad_MP, MountingHole:MountingHole_2.2mm_M2_ISO7380_Pad_TopOnly, F.Cu at (187.2, 21.0)
- added H2: MountingHole_Pad_MP, MountingHole:MountingHole_2.2mm_M2_ISO7380_Pad_TopOnly, F.Cu at (176.5, 18.5)
- added J5: 5-146278-6, 6 pin male header:TE_5-146278-6, F.Cu at (142.8, 88.7)
- added J6: PPTC061LFBN-RC, 6 pin female header:SULLINS_PPTC061LFBN-RC, F.Cu at (136.5, 95.0)
- added J7: 68000-103HLF, 3 pin male header:AMPHENOL_68000-103HLF, F.Cu at (142.8, 127.6)
- added J8: PPTC031LFBN-RC, footprints:CONN_PPTC031_SUL, F.Cu at (136.5, 130.2)
- added REF**: MountingHole_2.2mm_M2_Pad_Via, MountingHole:MountingHole_2.2mm_M2_Pad_Via, F.Cu at (64.0, 145.4)
- added REF**: MountingHole_3.2mm_M3_Pad_Via, MountingHole:MountingHole_3.2mm_M3_Pad_Via, F.Cu at (118.4, 88.1)
- added REF**: MountingHole_2.2mm_M2_Pad_Via, MountingHole:MountingHole_2.2mm_M2_Pad_Via, F.Cu at (101.5, 107.1)
- added REF**: MountingHole_2.2mm_M2_Pad_Via, MountingHole:MountingHole_2.2mm_M2_Pad_Via, F.Cu at (37.1, 88.4)
- added REF**: MountingHole_2.2mm_M2_Pad_Via, MountingHole:MountingHole_2.2mm_M2_Pad_Via, F.Cu at (135.3, 106.8)
- added REF**: MountingHole_2.2mm_M2_Pad_Via, MountingHole:MountingHole_2.2mm_M2_Pad_Via, F.Cu at (-7.48, 145.9)
- added REF**: MountingHole_2.2mm_M2_Pad_Via, MountingHole:MountingHole_2.2mm_M2_Pad_Via, F.Cu at (64.0, 88.4)
- added REF**: MountingHole_2.2mm_M2_Pad_Via, MountingHole:MountingHole_2.2mm_M2_Pad_Via, F.Cu at (-34.5, 145.9)
- added REF**: MountingHole_2.2mm_M2_Pad_Via, MountingHole:MountingHole_2.2mm_M2_Pad_Via, F.Cu at (37.1, 145.4)
- added RST: Jumper_2_Open, Jumper:SolderJumper-2_P1.3mm_Open_TrianglePad1.0x1.5mm, B.Cu at (149.0, 124.2)
- added boot: Jumper_2_Open, Jumper:SolderJumper-2_P1.3mm_Open_TrianglePad1.0x1.5mm, B.Cu at (163.4, 96.5)
- C1: value 10uf -> 1uf
- C11: value 150uf -> 10uf; footprint Capacitor_SMD:C_Elec_6.3x7.7 -> Capacitor_SMD:C_1812_4532Metric; moved to B.Cu
- C12, R23: moved to B.Cu
- C13: value 10uf -> 0.1uf; moved to B.Cu
- C14: value 10uf -> 1nf; moved to B.Cu
- C2: value 1uf -> 10uf; moved to F.Cu
- C3, C5, C9, TP4, TP5, TP6: moved to F.Cu
- C4: value 10uf -> BFC233820334; footprint Capacitor_SMD:C_1812_4532Metric -> x1 emi capacitor:CAPRR1500W80L1750T850H1500P; moved to F.Cu
- C6: value 10uf -> 0.1uf; moved to F.Cu
- C7: value 0.1uf -> 10uf; moved to F.Cu
- C8: value 0.1uf 275vac -> 150uf; footprint Capacitor_THT:C_Rect_L18.0mm_W6.0mm_P15.00mm_FKS3_FKP3 -> Capacitor_SMD:C_Elec_6.3x7.7
- J1, J2: footprint TerminalBlock_MetzConnect:TerminalBlock_MetzConnect_360271_1x01_Horizontal_ScrewM3.0_Boxed -> MountingHole:MountingHole_3mm_Pad_Via
- J3: value Screw_Terminal_01x01 -> 2013499-1; footprint TerminalBlock_MetzConnect:TerminalBlock_MetzConnect_360271_1x01_Horizontal_ScrewM3.0_Boxed -> usb micro:TE_2013499-1; moved to B.Cu
- PS1: value HLK-5M12 -> HLK-PM01; footprint Converter_ACDC:Converter_ACDC_Hi-Link_HLK-5Mxx -> hlk-pm01:CONV_HLK-PM01
- Q1: value NPN -> BTA16-600B; footprint Package_TO_SOT_SMD:SOT-23_Handsoldering -> Package_TO_SOT_THT:TO-220-3_Vertical
- R10: value 4.7k -> 1k
- R11, R12: value 1M -> 2.2K; moved to B.Cu
- R13: value 10k -> 22K; moved to B.Cu
- R14, R15: value 2.2K -> 1k; moved to B.Cu
- R16: value 1k -> 22K; moved to B.Cu
- R17: value 100k -> 2.2K; moved to B.Cu
- R18: value 1k -> 2.2K; moved to B.Cu
- R2: value 10k -> 4.7k
- R21: value 22K -> 220; moved to B.Cu
- R22: value 100k -> 4.7k; moved to B.Cu
- R6: value 4.7k -> 10k; moved to B.Cu
- R7, R8: value 1k -> 1M; moved to B.Cu
- R9: value 220 -> 1k
- TP1, TP7, TP8: footprint TestPoint:TestPoint_Pad_D4.0mm -> TestPoint:TestPoint_Pad_D2.5mm; moved to F.Cu
- TP10, TP16: footprint TestPoint:TestPoint_Pad_D4.0mm -> TestPoint:TestPoint_Pad_D2.5mm; moved to B.Cu
- TP2: value TestPoint -> TestPoint_Alt; footprint TestPoint:TestPoint_Pad_D4.0mm -> TestPoint:TestPoint_Pad_4.0x4.0mm; moved to F.Cu
- TP3: value TestPoint -> TestPoint_Alt; footprint TestPoint:TestPoint_Pad_D2.5mm -> TestPoint:TestPoint_Pad_4.0x4.0mm; moved to F.Cu
- TP9: footprint TestPoint:TestPoint_Pad_D4.0mm -> TestPoint:TestPoint_Pad_D2.5mm
- U1: value LM1117DT-3.3 -> L78M05ABDT-TR; footprint Package_TO_SOT_SMD:TO-252-3_TabPin2 -> PCM_JLCPCB:TO-252-2_L6.5-W6.1-P4.58-LS10.0-TL; moved to F.Cu
- U2: value L78M05ABDT-TR -> ESP32-C3-WROOM-02U; footprint PCM_JLCPCB:TO-252-2_L6.5-W6.1-P4.58-LS10.0-TL -> RF_Module:ESP32-C3-WROOM-02U
- U3: value ESP32-WROOM-32 -> LM1117DT-3.3; footprint RF_Module:ESP32-WROOM-32 -> Package_TO_SOT_SMD:TO-252-3_TabPin2; moved to F.Cu
- U4: value L78M05ABDT-TR -> PC817; footprint PCM_JLCPCB:TO-252-2_L6.5-W6.1-P4.58-LS10.0-TL -> Package_DIP:DIP-4_W7.62mm
- U5: value PC817 -> LM358DT; footprint Package_DIP:DIP-4_W7.62mm -> operational amplifier:SOIC127P600X175-8N; moved to B.Cu
- U6: value TLV9001IDCK -> ACS712xLCTR-20A; footprint Package_TO_SOT_SMD:SOT-353_SC-70-5 -> Package_SO:SOIC-8_3.9x4.9mm_P1.27mm; moved to B.Cu
- U7: value ACS712xLCTR-20A -> HCNR200-500E; footprint Package_SO:SOIC-8_3.9x4.9mm_P1.27mm -> high prescision optocoupler:OPTO_HCNR200-500E; moved to B.Cu
- moved C12 192.9 mm to (110.8, 133.6), turned to 90 degrees
- moved R12 176.3 mm to (121.8, 130.0)
- moved R11 175.5 mm to (121.8, 124.3)
- moved R23 173.7 mm to (116.5, 95.1), turned to -90 degrees
- moved R14 168.4 mm to (101.8, 85.6), turned to -90 degrees
- moved R21 168.1 mm to (154.8, 122.6), turned to -90 degrees
- moved C14 163.8 mm to (122.3, 99.1), turned to 180 degrees
- moved R15 162.5 mm to (107.5, 86.8)
- moved U7 161.6 mm to (118.3, 109.3), turned to -90 degrees
- moved U6 158.0 mm to (130.1, 98.6), turned to 180 degrees
- moved U4 146.7 mm to (99.5, 90.8)
- moved C13 145.8 mm to (123.3, 93.1), turned to 90 degrees
- moved C10 138.3 mm to (121.8, 119.6), turned to 180 degrees
- moved TP13 134.9 mm to (105.8, 133.3), turned to 180 degrees
- moved C11 130.7 mm to (121.8, 134.8), turned to 0 degrees
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Connections:
- C1 pad 1: VCC -> Net-(JP2-B)
- C10 pad 1: V5V2 -> Net-(C10-Pad1)
- C11 pad 1: VCC -> GND
- C11 pad 2: GND -> Net-(C11-Pad2)
- C12 pad 1: GND -> V5V_base
- C12 pad 2: Net-(C12-Pad2) -> GND
- C13 pad 1: Net-(C13-Pad1) -> V5V_base
- C14 pad 1: V5V -> Net-(U6-FILTER)
- C2 pad 1: Net-(U3-EN) -> VCC
- C3 pad 1: VCC -> V5V
- C4 pad 1: 3V3 -> Net-(PS1-AC1)
- C4 pad 2: GND -> /N
- C5 pad 1: V5V -> 3V3
- C7 pad 1: 3V3 -> VCC
- C8 pad 1: Net-(JP1-A) -> VCC_base
- C8 pad 2: /N -> GND
- C9 pad 1: VCC -> 3V3
- D4 pad 1: V5V2 -> V5V
- D4 pad 2: Net-(D4-DOUT) -> unconnected-(D4-DOUT-Pad2)
- F1 pad 1: /L -> /L2
- F1 pad 2: Net-(JP1-A) -> Net-(PS1-AC1)
- J3 pad 1: /communication -> VCC
- PS1 pad 1: Net-(JP1-B) -> Net-(PS1-AC1)
- PS1 pad 2: Net-(JP2-B) -> /N
- PS1 pad 4: VCC -> VCC_base
- Q1 pad 1: Net-(Q1-C) -> /L3
- Q1 pad 2: Net-(Q1-B) -> /L2
- Q1 pad 3: GND -> /triac in
- R1 pad 2: Net-(D1-A) -> Net-(JP2-B)
- R10 pad 1: Net-(Q1-C) -> /switch_base
- R10 pad 2: Net-(Q2-B) -> Net-(R10-Pad2)
- R11 pad 1: Net-(C12-Pad2) -> /in-
- R11 pad 2: /L -> Net-(C10-Pad1)
- R12 pad 1: Net-(C13-Pad1) -> /in+
- R12 pad 2: /N -> Net-(C11-Pad2)
- R13 pad 1: V5V2 -> V5V_base
- R13 pad 2: Net-(Q1-C) -> /in+
- R14 pad 1: /in+ -> Net-(R14-Pad1)
- R14 pad 2: Net-(C12-Pad2) -> /triac in
- R15 pad 1: /in- -> /triac in
- R15 pad 2: Net-(C13-Pad1) -> GND
- R16 pad 1: Net-(R16-Pad1) -> Net-(U5-OUT1)
- R16 pad 2: /triac in -> /in-
- R17 pad 1: Net-(Q1-C) -> /V_isolation
- R17 pad 2: Net-(Q3-G) -> Net-(U5-OUT1)
- R18 pad 1: /triac in -> /V_isolation
- R2 pad 1: 3V3 -> Net-(U2-IO7)
- R2 pad 2: Net-(U3-EN) -> Net-(D1-A)
- R21 pad 1: Net-(R21-Pad1) -> /ring light
- R21 pad 2: /in- -> Net-(D4-DIN)
- R22 pad 1: GND -> Net-(R22-Pad1)
- R22 pad 2: V5V -> /V_isolation
- R23 pad 1: /V_isolation -> V5V_base
- R23 pad 2: Net-(R21-Pad1) -> Net-(R23-Pad2)
- R3 pad 2: Net-(U3-IO0) -> /boot
- R6 pad 1: /defacto_en -> V5V
- R6 pad 2: Net-(Q1-B) -> Net-(D3-A)
- R7 pad 1: V5V -> Net-(C10-Pad1)
- R7 pad 2: /button in -> /N
- R8 pad 1: /switch  -> Net-(C11-Pad2)
- R8 pad 2: Net-(R8-Pad2) -> /L
- R9 pad 1: /ring light -> V5V
- R9 pad 2: Net-(D4-DIN) -> /button in
- RV1 pad 1: Net-(JP1-A) -> /N
- RV1 pad 2: /N -> Net-(PS1-AC1)
- TP10 pad 1: /N -> /in-
- TP11 pad 1: /AN XS1 -> /in+
- TP12 pad 1: /AN XS2 -> /triac in
- TP13 pad 1: /DIG XS -> /V_isolation
- TP15 pad 1: /XTAL OUT -> /current_sense
- TP16 pad 1: Net-(JP1-B) -> /Volt_sense
- TP2 pad 1: VCC -> /L3
- TP3 pad 1: Net-(U3-SDO/SD0) -> /N
- TP4 pad 1: Net-(U3-SDI/SD1) -> /XTAL OUT
- TP5 pad 1: Net-(U3-SCK/CLK) -> V5V
- TP6 pad 1: Net-(U3-SCS/CMD) -> Net-(U2-IO8)
- TP7 pad 1: 3V3 -> Net-(U2-IO9)
- TP8 pad 1: V5V -> VCC
- TP9 pad 1: Net-(JP1-A) -> 3V3
- U1 pad 1: GND -> VCC
- U1 pad 3: VCC -> V5V
- U2 pad 1: VCC -> 3V3
- U2 pad 3: V5V -> /V_sense
- U2 pad 4: GND -> /switch 
- U3 pad 3: Net-(U3-EN) -> VCC
- U4 pad 1: VCC -> Net-(R10-Pad2)
- U4 pad 3: V5V2 -> Net-(R14-Pad1)
- U4 pad 4: GND -> V5V_base
- U5 pad 1: Net-(R8-Pad2) -> Net-(U5-OUT1)
- U5 pad 2: GND -> /in-
- U5 pad 3: Net-(R16-Pad1) -> /in+
- U5 pad 4: V5V2 -> GND
- U6 pad 1: /in+ -> /L
- U6 pad 2: GND -> /L
- U6 pad 3: /in- -> /L2
- U6 pad 4: Net-(R21-Pad1) -> /L2
- U6 pad 5: V5V -> GND
- U7 pad 1: /L -> GND
- U7 pad 2: /L -> Net-(R22-Pad1)
- U7 pad 3: /N -> /Volt_sense
- U7 pad 4: /N -> Net-(R23-Pad2)
- U7 pad 5: GND -> /in+
- U7 pad 6: Net-(U7-FILTER) -> /in-
- U7 pad 7: /I_sense -> (no net)
- U7 pad 8: V5V -> (no net)
Routing:
- net /in+: track 0.00 -> 26.5 mm
- net Net-(JP2-B): track 0.00 -> 23.9 mm
- net /in-: track 0.00 -> 23.4 mm
- net /button in: track 0.00 -> 20.4 mm
- net Net-(U5-OUT1): track 0.00 -> 19.0 mm
- net /USB_D-: track 0.00 -> 14.4 mm
- net /USB_D+: track 0.00 -> 14.4 mm
- net Net-(J4-Pin_3): track 0.00 -> 12.7 mm
- net Net-(J4-Pin_2): track 0.00 -> 12.6 mm
- net Net-(U2-IO7): track 0.00 -> 10.8 mm
- net Net-(C11-Pad2): track 0.00 -> 7.69 mm
- net Net-(C10-Pad1): track 0.00 -> 7.59 mm
- net Net-(D4-DIN): track 0.00 -> 6.80 mm
- net /boot: track 0.00 -> 6.04 mm
- net /ring light: track 0.00 -> 5.26 mm
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Other:
- board size 69.9 x 69.6 mm -> 205 x 69.2 mm
- copper layers 2 -> 4
