File: easy home electronics.kicad_sch (KiCad schematic)
At the start: 109 parts, among them J1 Screw_Terminal_01x01, J2 Screw_Terminal_01x01, J3 Screw_Terminal_01x01, J4 Conn_01x04_Pin, Q1 NPN, Q2 NPN, Q3 PMOS, Q4 NPN, Q5 BTA16-600B, Q6 NPN, SW1 SW_Push, SW2 SW_Push, SW3 SW_Push, U1 LM1117DT-3.3, U2 L78M05ABDT-TR, U3 ESP32-WROOM-32, U4 L78M05ABDT-TR, U5 PC817, U6 TLV9001IDCK, U7 ACS712xLCTR-20A, U8 HCNR200-500E

Commit message: Add files via upload
new design backup
Parts:
- removed C13, C14, C9: 10uf, Capacitor_SMD:C_1812_4532Metric, symbol Device:C
- removed C15: 22uf, Capacitor_SMD:C_1812_4532Metric, symbol Device:C
- removed C2: 1uf, Capacitor_SMD:C_1812_4532Metric, symbol Device:C
- removed C7: 0.1uf, Capacitor_SMD:C_1812_4532Metric, symbol Device:C
- removed D5, D6, D7: WS2812B, LED_SMD:LED_WS2812B_PLCC4_5.0x5.0mm_P3.2mm, symbol LED:WS2812B
- removed J3: Screw_Terminal_01x01, TerminalBlock_MetzConnect:TerminalBlock_MetzConnect_360271_1x01_Horizontal_ScrewM3.0_Boxed, symbol Connector:Screw_Terminal_01x01
- removed JP1, JP2: SolderJumper_2_Open, Jumper:SolderJumper-2_P1.3mm_Open_RoundedPad1.0x1.5mm, symbol Jumper:SolderJumper_2_Open
- removed L1: L_Coupled_1243, Inductor_THT:Choke_Schaffner_RN212-04-12.5x18.0mm, symbol Device:L_Coupled_1243
- removed PS1: HLK-5M12, Converter_ACDC:Converter_ACDC_Hi-Link_HLK-5Mxx, symbol Converter_ACDC:HLK-5M12
- removed Q1, Q2, Q4, Q6: NPN, Package_TO_SOT_SMD:SOT-23_Handsoldering, symbol Simulation_SPICE:NPN
- removed Q3: PMOS, Package_TO_SOT_SMD:SOT-23_Handsoldering, symbol Simulation_SPICE:PMOS
- removed R10, R5: 4.7k, Resistor_SMD:R_1812_4532Metric_Pad1.30x3.40mm_HandSolder, symbol Device:R
- removed R14, R15, R23, R24: 2.2K, Resistor_SMD:R_1812_4532Metric_Pad1.30x3.40mm_HandSolder, symbol Device:R
- removed R19, R21: 22K, Resistor_SMD:R_1812_4532Metric_Pad1.30x3.40mm_HandSolder, symbol Device:R
- removed R20, R22: 100k, Resistor_SMD:R_1812_4532Metric_Pad1.30x3.40mm_HandSolder, symbol Device:R
- removed R4: 10k, Resistor_SMD:R_1812_4532Metric_Pad1.30x3.40mm_HandSolder, symbol Device:R
- removed SW1, SW2: SW_Push, Button_Switch_THT:SW_PUSH_6mm_H5mm, symbol Switch:SW_Push
- removed TP14, TP3: TestPoint, TestPoint:TestPoint_Pad_D2.5mm, symbol Connector:TestPoint
- removed TP17, TP18, TP19, TP2, TP20, TP21, TP22, TP23, TP24, TP25, TP26, TP27, TP29, TP30: TestPoint, TestPoint:TestPoint_Pad_D4.0mm, symbol Connector:TestPoint
- removed U3: ESP32-WROOM-32, RF_Module:ESP32-WROOM-32, symbol RF_Module:ESP32-WROOM-32
- removed U4: L78M05ABDT-TR, PCM_JLCPCB:TO-252-2_L6.5-W6.1-P4.58-LS10.0-TL, symbol PCM_JLCPCB-Power:LDO, 5V, 0.5A
- removed U6: TLV9001IDCK, Package_TO_SOT_SMD:SOT-353_SC-70-5, symbol Amplifier_Operational:TLV9001IDCK
- removed U8: HCNR200-500E, Package_DIP:DIP-8_W7.62mm, symbol HCNR200-500E:HCNR200-500E
- added C1: 1uf, Capacitor_SMD:C_1812_4532Metric, symbol Device:C
- added C4: BFC233820334, x1 emi capacitor:CAPRR1500W80L1750T850H1500P, symbol BFC233820334:BFC233820334
- added C5: 10uf, Capacitor_SMD:C_1812_4532Metric, symbol Device:C
- added J3: 2013499-1, usb micro:TE_2013499-1, symbol 2013499-1:2013499-1
- added J5: 5-146278-6, 6 pin male header:TE_5-146278-6, symbol 5-146278-6:5-146278-6
- added J6: PPTC061LFBN-RC, 6 pin female header:SULLINS_PPTC061LFBN-RC, symbol PPTC061LFBN-RC:PPTC061LFBN-RC
- added J7: 68000-103HLF, 3 pin male header:AMPHENOL_68000-103HLF, symbol 68000-103HLF:68000-103HLF
- added J8: PPTC031LFBN-RC, footprints:CONN_PPTC031_SUL, symbol 2025-07-05_06-44-57:PPTC031LFBN-RC
- added JP1, JP2: Jumper_2_Open, Jumper:SolderJumper-2_P1.3mm_Open_TrianglePad1.0x1.5mm, symbol Jumper:Jumper_2_Open
- added PS1: HLK-PM01, hlk-pm01:CONV_HLK-PM01, symbol HLK-PM01:HLK-PM01
- added R16: 22K, Resistor_SMD:R_1812_4532Metric_Pad1.30x3.40mm_HandSolder, symbol Device:R
- added R18: 2.2K, Resistor_SMD:R_1812_4532Metric_Pad1.30x3.40mm_HandSolder, symbol Device:R
- added R7, R8: 1M, Resistor_SMD:R_1812_4532Metric_Pad1.30x3.40mm_HandSolder, symbol Device:R
- added TP2, TP3: TestPoint_Alt, TestPoint:TestPoint_Pad_4.0x4.0mm, symbol Connector:TestPoint_Alt
- added U2: ESP32-C3-WROOM-02U, RF_Module:ESP32-C3-WROOM-02U, symbol RF_Module:ESP32-C3-WROOM-02U
- added U5: LM358DT, operational amplifier:SOIC127P600X175-8N, symbol LM358DT:LM358DT
- added U7: HCNR200-500E, high prescision optocoupler:OPTO_HCNR200-500E, symbol HCNR200-500E:HCNR200-500E
- C11: value 150uf -> 10uf; footprint Capacitor_SMD:C_Elec_6.3x7.7 -> Capacitor_SMD:C_1812_4532Metric
- C6: value 10uf -> 0.1uf
- C8: value 0.1uf 275vac -> 150uf; footprint Capacitor_THT:C_Rect_L18.0mm_W6.0mm_P15.00mm_FKS3_FKP3 -> Capacitor_SMD:C_Elec_6.3x7.7
- J1, J2: footprint TerminalBlock_MetzConnect:TerminalBlock_MetzConnect_360271_1x01_Horizontal_ScrewM3.0_Boxed -> MountingHole:MountingHole_3mm_Pad_Via
- R11, R12: value 1M -> 2.2K
- R13: value 10k -> 22K
- R17: value 100k -> 2.2K
- R19: renamed from R25; now not fitted
- R2: value 10k -> 4.7k
- R20: renamed from R26; now not fitted
- R6: value 4.7k -> 10k
- TP1, TP10, TP16, TP7, TP8, TP9: footprint TestPoint:TestPoint_Pad_D4.0mm -> TestPoint:TestPoint_Pad_D2.5mm
- TP14: renamed from TP28; now not fitted
- renumbered C16 to C13, C17 to C14, C3 to C2, C5 to C3, C1 to C7, C4 to C9, Q5 to Q1, R8 to R10, R16 to R14, R18 to R15, R9 to R21, R27 to R22, R28 to R23, R7 to R9, U2 to U1, U1 to U3, U5 to U4, U7 to U6
Connections:
- net AN XS1 is gone; now on net in+: TP11.1
- net AN XS2 is gone; now on net triac in: TP12.1
- net DIG XS is gone; now on net V_isolation: TP13.1
- net defacto_en is gone; now on net V5V: R6.1
- net 3V3: now also TP9.1, C5.1, U2.1 (3V3); no longer R2.1, TP7.1
- net GND: now also C11.1, C12.2, C8.2, C1.2, C5.2, J3.5 (GND), J5.2, J5.4, J5.6, J6.2, J6.4, J6.6, J7.3, J8.3, JP1.1 (A), JP2.1 (A), PS1.3 (-VO), R18.2, U2.19 (GND), U2.9 (GND), U5.4 (VCC-), U7.1; no longer C11.2, C12.1
- net I_sense: now also J5.1, U2.15 (IO3); no longer U6.7 (VIOUT)
- net L: now also R8.2; no longer F1.1, Q1.2 (A2), R11.2
- net L_sense: now also U2.16 (IO2)
- net N: now also RV1.1, C4.2, PS1.2 (AC2), R7.2, TP3.1; no longer C8.2, Q1.1 (A1), R12.2, RV1.2, TP10.1, U6.3 (IP-), U6.4 (IP-)
- net V5V: now also D4.1 (VDD), TP5.1, J7.1, U5.8 (VCC+); no longer C13.1, R23.1, TP8.1, U6.8 (VCC)
- net VCC: now also TP8.1, J3.1 (VBUS), J7.2; no longer C11.1
- net V_isolation: now also R17.1, R18.1
- net V_sense: now also J5.3, U2.3 (IO4)
- net XTAL OUT: now also TP4.1, U2.17 (IO1); no longer TP15.1
- net button in: now also U2.10 (IO10)
- net in+: now also R12.1, R13.2, U5.3 (IN1+), U7.5
- net in-: now also R11.1, TP10.1, R16.2, U5.2 (IN1-), U7.6
- net ring light: now also U2.5 (IO6)
- net switch : now also J5.5, U2.4 (IO5); no longer R10.1
- net at J4.2 (Pin_2): now also U2.11 (IO20/RXD)
- net at J4.3 (Pin_3): now also U2.12 (IO21/TXD)
- net boot: now reaches R3.2
- net boot: now also JP1.2 (B), U2.18 (IO0)
- net at R2.2: now also D1.2 (A)
- net Volt_sense: now reaches TP16.1
- net Volt_sense: now also J6.3, U7.3
- net at R17.2: now also R16.1, U5.1 (OUT1)
- net at D3.2 (A): now also R6.2
- net at TP6.1: now also U2.7 (IO8)
- net at R1.2: now also C1.1, JP2.2 (B), U2.2 (EN); no longer D1.2 (A)
- net at R22.1: now also U7.2
- net at R23.2: now also U7.4
- net V5V2 renamed V5V_base
- net V5V_base: now also C12.1, C13.1, R23.1, U6.8 (VCC), J8.1; no longer C10.1, D4.1 (VDD)
- new net: TP7.1, U2.8 (IO9)
- new net: C4.1, F1.2, PS1.1 (AC1), RV1.2
- new net: R2.1, U2.6 (IO7)
- new net: C11.2, R12.2, R8.1
- new net: C10.1, R11.2, R7.1
- new net: J3.SH1 (SHIELD), J3.SH2 (SHIELD), J3.SH3 (SHIELD), J3.SH4 (SHIELD), J3.SH5 (SHIELD), J3.SH6 (SHIELD)
- new net L2: F1.1, Q1.2 (A2), U6.3 (IP-), U6.4 (IP-)
- new net L3: Q1.1 (A1), TP2.1
- new net USB_D+: J3.3 (DP), U2.14 (IO19)
- new net USB_D-: J3.2 (DN), U2.13 (IO18)
- new net VCC_base: C8.1, J8.2, PS1.4 (+VO)
- new net current_sense: J6.1, TP15.1, U6.7 (VIOUT)
- new net switch_base: J6.5, R10.1
- no-connect marks 11 -> 6
Other:
- note added: "3 pin female connector on power board"
- note added: "3 pin male connector on logic board"
- note added: "6 pin female connector on power board"
- note added: "6 pin male connector on logic board"
- note added: "BOARD CONNECTORS"
- note added: "female"
- note added: "led light"
- note added: "male"
- note removed: "controller section"
- note removed: "defacto switching system incase of MCU fault"
- note removed: "enable input"
- note removed: "led ring light around switch"
- note removed: "to triac"
- title: (none) -> EASY HOME ELECTRONICS
- moved on the sheet: C13, C14, C2, C3, C7, C9, D4, Q1, R10, R14, R15, R21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
